File: cap_array_rx/cap_array_rx.kicad_pcb (KiCad board)
At the start: 4 copper layers, 44 parts, among them CN1 B4B-PH-K-S, J1 SWIO, J10 Conn_01x01, J11 Conn_01x01, J12 Conn_01x01, J13 Conn_01x01, J14 Conn_01x01, J15 Conn_01x01, J16 Conn_01x01, J17 Conn_01x01, J18 Conn_01x01, J2 NRST, J3 Conn_01x01, J4 Conn_01x01, J5 Conn_01x01, J6 Conn_01x01, J7 Conn_01x01, J8 Conn_01x01, J9 Conn_01x01, U1 CH32V003F4P6, U2 AP2112K-3.3TRG1, U4 OPA2356AIDGKR, U5 TLV3501AIDBVR

Commit message: Initial commit: Nesting project files under capacitance subdirectory
Parts:
- removed R2: 100, Resistor_SMD:R_0805_2012Metric_Pad1.20x1.40mm_HandSolder
- added C10: 2.2 pF, Capacitor_SMD:C_0805_2012Metric_Pad1.18x1.45mm_HandSolder, F.Cu at (76.5, 70.5)
- added D2: BZT52C3V3, EasyEDA:SOD-123_L2.7-W1.6-LS3.7-RD, F.Cu at (65.5, 83.5)
- JP1, JP2, JP3: moved to B.Cu
- R1: value 1 k -> 2.2 K
- R3: value 1 K -> 1.2 k
- R4: value 100 -> 1 k
- moved C2 56.0 mm to (49.0, 64.0), turned to 90 degrees
- moved C4 54.3 mm to (52.0, 60.0)
- moved CN1 51.9 mm to (50.0, 69.0)
- moved U2 51.9 mm to (52.0, 63.5)
- moved C5 48.1 mm to (57.0, 71.5), turned to -90 degrees
- moved C6 45.3 mm to (60.0, 72.5), turned to 180 degrees
- moved C9 44.6 mm to (60.0, 65.0), turned to 0 degrees
- moved J7 42.8 mm to (69.5, 84.6)
- moved J8 42.5 mm to (69.5, 91.3)
- moved J9 42.1 mm to (69.5, 98.0)
- moved J10 41.9 mm to (69.5, 104.7)
- moved C8 39.7 mm to (60.0, 67.5), turned to 0 degrees
- moved JP1 39.7 mm to (61.8, 80.2)
- moved JP2 39.7 mm to (61.8, 79.2)
- moved JP3 39.7 mm to (61.8, 78.2)
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Connections:
- D1 pad 2: GND -> v_half_ref
- R1 pad 2: Net-(U4-INA-) -> D
- R4 pad 2: GND -> v_half_ref
- R6 pad 1: +3.3V -> +5V
- R6 pad 2: Net-(U5--IN) -> v_half_ref
- R7 pad 1: Net-(U5--IN) -> v_half_ref
- U4 pad 2: Net-(U4-INA-) -> D
- U4 pad 3: D -> v_half_ref
- U4 pad 8: +3.3V -> +5V
- U5 pad 1: Net-(U5--IN) -> v_half_ref
- U5 pad 4: +3.3V -> +5V
- U5 pad 6: +3.3V -> +5V
Routing:
- net PC4: track 0.38 -> 58.8 mm, vias 0 -> 3
- net PC5: track 0.00 -> 50.5 mm, vias 0 -> 3
- net PC0: track 0.00 -> 42.3 mm, vias 0 -> 3
- net PC6: track 0.00 -> 40.1 mm, vias 0 -> 2
- net PC7: track 0.00 -> 28.6 mm, vias 0 -> 2
- net Net-(J14-Pin_1): track 0.00 -> 27.5 mm
- net Net-(J10-Pin_1): track 0.00 -> 26.5 mm
- net v_half_ref: track 0.00 -> 26.3 mm
- net +3.3V: track 0.00 -> 25.6 mm
- net PD3: track 0.00 -> 23.4 mm, vias 0 -> 2
- net GND: track 0.00 -> 22.1 mm, vias 0 -> 14
- net Net-(J9-Pin_1): track 0.00 -> 21.0 mm
- net Net-(J13-Pin_1): track 0.00 -> 20.2 mm
- net Net-(J15-Pin_1): track 0.00 -> 18.8 mm
- net Net-(J3-Pin_1): track 0.00 -> 17.1 mm
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- added copper zone on In2.Cu, net +5V
- added copper zone on In1.Cu, net GND
Other:
- board outline added: 57.5 x 56 mm

Commit message: with douple spi connection
Parts:
- added CN2: B4B-PH-K-S, EasyEDA:CONN-TH_B4B-PH-K-S, F.Cu at (50.0, 67.3)
- moved CN1 3.32 mm to (50.0, 72.3)
- moved C2 2.24 mm to (50.4, 62.3)
- moved C4 2.24 mm to (53.4, 58.3)
- moved U2 2.24 mm to (53.4, 61.8)
- moved J1 1.71 mm to (52.5, 78.7)
- moved C7 1.69 mm to (58.6, 71.5), turned to -90 degrees
- moved C6 1.41 mm to (61.0, 71.5), turned to -90 degrees
- moved C5 0.75 mm to (56.2, 71.5)
Routing:
- net SCL: track 15.2 -> 18.8 mm
- net SDA: track 12.9 -> 16.5 mm
- net GND: track 22.1 -> 22.8 mm
- net Net-(J1-Pin_1): track 7.96 -> 7.25 mm
- net +5V: track 13.4 -> 14.0 mm
- net +3.3V: track 25.6 -> 26.3 mm

Commit message: Modular Design
Parts:
- removed the C3 at (68.5, 81.0)
- removed D2: BZT52C3V3, EasyEDA:SOD-123_L2.7-W1.6-LS3.7-RD
- removed the R5 at (68.5, 79.0)
- added C10: 100 nF, Capacitor_SMD:C_0805_2012Metric_Pad1.18x1.45mm_HandSolder, F.Cu at (75.7, 65.2)
- added C11: 1 nF, Capacitor_SMD:C_0805_2012Metric_Pad1.18x1.45mm_HandSolder, F.Cu at (66.0, 76.2)
- added C8: 1000 pF, Capacitor_SMD:C_0805_2012Metric_Pad1.18x1.45mm_HandSolder, F.Cu at (72.2, 71.5)
- added Q1: 2N7002, Package_TO_SOT_SMD:SOT-23, F.Cu at (55.8, 85.0)
- added R10: 1k, Resistor_SMD:R_0805_2012Metric, F.Cu at (66.0, 74.0)
- added R11: 200, Resistor_SMD:R_0805_2012Metric, F.Cu at (66.2, 83.2)
- added R12: 1 k, Resistor_SMD:R_0805_2012Metric, F.Cu at (69.5, 67.5)
- added R2: 100 k, Resistor_SMD:R_0805_2012Metric, F.Cu at (76.0, 71.5)
- added R7: 620, Resistor_SMD:R_0805_2012Metric, F.Cu at (72.1, 82.5)
- added R8: 100 k, Resistor_SMD:R_0805_2012Metric, F.Cu at (72.0, 84.8)
- added R9: 200, Resistor_SMD:R_0805_2012Metric, F.Cu at (66.2, 81.2)
- added TP1: TestPoint_2Pole, TestPoint:TestPoint_2Pads_Pitch2.54mm_Drill0.8mm, F.Cu at (73.5, 74.2)
- added TP2: TestPoint_2Pole, TestPoint:TestPoint_2Pads_Pitch2.54mm_Drill0.8mm, F.Cu at (69.5, 74.0)
- added TP3: TestPoint, Connector_Pin:Pin_D0.7mm_L6.5mm_W1.8mm_FlatFork, F.Cu at (68.8, 86.8)
- added TP4: TestPoint, Connector_Pin:Pin_D0.7mm_L6.5mm_W1.8mm_FlatFork, F.Cu at (75.8, 83.5)
- added TP5: TestPoint, Connector_Pin:Pin_D0.7mm_L6.5mm_W1.8mm_FlatFork, F.Cu at (65.2, 78.8)
- added TP6: TestPoint, Connector_Pin:Pin_D0.7mm_L6.5mm_W1.8mm_FlatFork, F.Cu at (62.2, 71.8)
- C1: renamed from C8; footprint Capacitor_SMD:C_0805_2012Metric_Pad1.18x1.45mm_HandSolder -> Capacitor_SMD:C_0603_1608Metric
- C2: renamed from C9; footprint Capacitor_SMD:C_0805_2012Metric_Pad1.18x1.45mm_HandSolder -> Capacitor_SMD:C_0603_1608Metric
- C3: renamed from C7; footprint Capacitor_SMD:C_0805_2012Metric_Pad1.18x1.45mm_HandSolder -> Capacitor_SMD:C_0603_1608Metric
- C4: renamed from C5; footprint Capacitor_SMD:C_0805_2012Metric_Pad1.18x1.45mm_HandSolder -> Capacitor_SMD:C_0603_1608Metric
- C5: renamed from C6; footprint Capacitor_SMD:C_0805_2012Metric_Pad1.18x1.45mm_HandSolder -> Capacitor_SMD:C_0603_1608Metric
- C7: renamed from C10; value 2.2 pF -> 1.5 pF
- R1: value 2.2 K -> 10 k; footprint Resistor_SMD:R_0805_2012Metric_Pad1.20x1.40mm_HandSolder -> Resistor_SMD:R_0805_2012Metric
- R3: value 1.2 k -> 10 k; footprint Resistor_SMD:R_0805_2012Metric_Pad1.20x1.40mm_HandSolder -> Resistor_SMD:R_0805_2012Metric
- R4: footprint Resistor_SMD:R_0805_2012Metric_Pad1.20x1.40mm_HandSolder -> Resistor_SMD:R_0805_2012Metric
- R5: renamed from R6; footprint Resistor_SMD:R_0805_2012Metric_Pad1.20x1.40mm_HandSolder -> Resistor_SMD:R_0805_2012Metric
- R6: renamed from R7; footprint Resistor_SMD:R_0805_2012Metric_Pad1.20x1.40mm_HandSolder -> Resistor_SMD:R_0805_2012Metric
- moved J6 21.7 mm to (47.8, 103.5), turned to -90 degrees
- moved J9 18.9 mm to (67.9, 103.5), turned to -90 degrees
- moved C9 16.1 mm to (51.2, 74.2), turned to -90 degrees
- moved J7 16.0 mm to (54.5, 103.5), turned to -90 degrees
- moved J8 14.8 mm to (61.2, 103.5), turned to -90 degrees
- moved U1 13.7 mm to (47.8, 74.2), turned to -90 degrees
- moved CN2 12.6 mm to (50.2, 54.8)
- moved CN1 12.1 mm to (50.2, 60.2)
- moved J2 11.2 mm to (99.0, 102.5)
- moved J4 11.2 mm to (99.0, 89.2)
- moved J5 11.2 mm to (99.0, 82.5)
- moved J3 11.2 mm to (99.0, 95.8)
- moved C1 10.4 mm to (57.0, 57.5), turned to 90 degrees
- moved J1 9.86 mm to (53.5, 78.5)
- moved C6 9.39 mm to (47.7, 71.2), turned to 0 degrees
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- renumbered C2 to C6, C4 to C9, J2 to J1, J11 to J10, J12 to J11, J13 to J12, J14 to J13, J15 to J14, J16 to J15, J17 to J16, J18 to J17, J1 to J18, J3 to J2, J4 to J3, J5 to J4, J6 to J5, J10 to J6, J9 to J7, J7 to J9, U2 to U1, U4 to U2, U1 to U3, U5 to U4
Connections:
- D1 pad 3: PA1 -> /PD2 Pre
- U2 pad 5: OUT_A -> Net-(U2-INB+)
- U3 pad 13: unconnected-(U1-PC3/T1CH3/T1CH1N_/UCTS_-Pad13) -> PC3
- U3 pad 19: unconnected-(U1-PD2/A3/T1CH1/T2CH3_/T1CH2N_-Pad19) -> PD2
- U3 pad 5: PA1 -> Net-(U3-PA1/OSCI/A1/T1CH2/OPN0)
- U4 pad 1: v_half_ref -> Net-(U4--IN)
- U4 pad 5: PD3 -> Net-(U4-OUT)
Routing:
- net v_half_ref: track 26.3 -> 70.8 mm, vias 0 -> 3
- net PC4: track 58.8 -> 31.4 mm, vias 3 -> 1
- net Net-(Q1-D): track 0.00 -> 25.8 mm, vias 0 -> 2
- net +5V: track 14.0 -> 38.8 mm, vias 8 -> 5
- net SCL: track 18.8 -> 40.3 mm
- net SDA: track 16.5 -> 38.0 mm
- net Net-(J8-Pin_1): track 15.4 -> 35.2 mm
- net Net-(J9-Pin_1): track 10.3 -> 29.8 mm
- net PD3: track 23.4 -> 4.54 mm, vias 2 -> 0
- net Net-(J7-Pin_1): track 21.0 -> 39.0 mm
- net Net-(J6-Pin_1): track 26.5 -> 43.6 mm
- net /PD2 Pre: track 0.00 -> 13.9 mm
- net Net-(U2-INB-): track 4.68 -> 17.3 mm
- net PC6: track 40.1 -> 28.9 mm
- net +3.3V: track 26.3 -> 15.6 mm
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