File: cap_array_rx/cap_array_rx.kicad_sch (KiCad schematic)
At the start: 45 parts, among them CN1 B4B-PH-K-S, J1 SWIO, J10 Conn_01x01, J11 Conn_01x01, J12 Conn_01x01, J13 Conn_01x01, J14 Conn_01x01, J15 Conn_01x01, J16 Conn_01x01, J17 Conn_01x01, J18 Conn_01x01, J2 NRST, J3 Conn_01x01, J4 Conn_01x01, J5 Conn_01x01, J6 Conn_01x01, J7 Conn_01x01, J8 Conn_01x01, J9 Conn_01x01, U1 CH32V003F4P6, U2 AP2112K-3.3TRG1, U4 OPA2356AIDGKR, U5 TLV3501AIDBVR

Commit message: with douple spi connection
Parts:
- added CN2: B4B-PH-K-S, EasyEDA:CONN-TH_B4B-PH-K-S, symbol EasyEDA:B4B-PH-K-S
- J1, J10, J11, J12, J13, J14, J15, J16, J17, J18, J2, J3, J4, J5, J6, J7, J8, J9, JP1, JP2, JP3: now left out of the parts list
Connections:
- net +5V: now also CN2.1
- net GND: now also CN2.2
- net SCL: now also CN2.4
- net SDA: now also CN2.3
Other:
- moved on the sheet: CN1

Commit message: version wiouth diodes to maximize capacitance re thinking envolope, simulation teste on openems available and configured
Parts:
- removed C3: 100 pF, Capacitor_SMD:C_0805_2012Metric_Pad1.18x1.45mm_HandSolder, symbol Device:C
- removed D1: BAT54SLT1G, EasyEDA:SOT-23_L2.9-W1.3-P1.90-LS2.4-BR, symbol EasyEDA:BAT54SLT1G
- removed D2: BZT52C3V3, EasyEDA:SOD-123_L2.7-W1.6-LS3.7-RD, symbol EasyEDA:BZT52C3V3
- removed R5: 10 K, Resistor_SMD:R_0805_2012Metric_Pad1.20x1.40mm_HandSolder, symbol Device:R
- added C10, C8: 100 pF, Capacitor_SMD:C_0805_2012Metric_Pad1.18x1.45mm_HandSolder, symbol Device:C
- added R2, R8: 100 k, Resistor_SMD:R_0805_2012Metric_Pad1.20x1.40mm_HandSolder, symbol Device:R
- added R7: 620, Resistor_SMD:R_0805_2012Metric_Pad1.20x1.40mm_HandSolder, symbol Device:R
- added R9: 1 k, Resistor_SMD:R_0805_2012Metric_Pad1.20x1.40mm_HandSolder, symbol Device:R
- added TP1: TestPoint_2Pole, symbol Connector:TestPoint_2Pole
- added TP2: TestPoint, symbol Connector:TestPoint
- C7: renamed from C10; value 2.2 pF -> 1.5 pF
- R1: value 2.2 K -> 4.7 k
- R3: value 1.2 k -> 10 k
- renumbered C8 to C1, C9 to C2, C7 to C3, C5 to C4, C6 to C5, C2 to C6, C4 to C9, J2 to J1, J11 to J10, J12 to J11, J13 to J12, J14 to J13, J15 to J14, J16 to J15, J17 to J16, J18 to J17, J1 to J18, J3 to J2, J4 to J3, J5 to J4, J6 to J5, J10 to J6, J9 to J7, J7 to J9, R6 to R5, R7 to R6, U2 to U1, U4 to U2, U1 to U3, U5 to U4
Connections:
- net +5V: now also R8.2
- net GND: now also C10.2
- net OUT_A: now also C8.2; no longer U2.5 (INB+)
- net PD3: now also R9.2; no longer U4.5 (OUT)
- net v_half_ref: now also C10.1, R2.1, R7.1; no longer U4.1 (-IN)
- net PA1: no longer names the net of U3.5 (PA1/OSCI/A1/T1CH2/OPN0)
- new net: C8.1, R2.2, U2.5 (INB+)
- new net: R9.1, U4.5 (OUT)
- new net: R7.2, R8.1, U4.1 (-IN)
- no-connect marks 5 -> 6
Other:
- moved on the sheet: C1, C2, C3, C4, C5, C6, C7, C9, CN2, R1, R3, R4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

Commit message: Modular Design
Parts:
- removed CN2: B4B-PH-K-S, EasyEDA:CONN-TH_B4B-PH-K-S, symbol EasyEDA:B4B-PH-K-S
- removed J10, J11, J12, J13, J14, J15, J16, J17, J2, J3, J4, J5, J6, J7, J8, J9: Conn_01x01, Connector_PinHeader_2.54mm:PinHeader_1x01_P2.54mm_Vertical, symbol Connector_Generic:Conn_01x01
- removed Mux_x1, Mux_y1: MUX508IDR, EasyEDA:SOIC-16_L9.9-W3.9-P1.27-LS6.0-BL, symbol EasyEDA:MUX508IDR
- removed TP2: TestPoint, symbol Connector:TestPoint
- removed U2: OPA2356AIDGKR, EasyEDA:VSSOP-8_L3.0-W3.0-P0.65-LS5.0-BL, symbol EasyEDA:OPA2356AIDGKR
- removed U3: CH32V003F4P6, EasyEDA:TSSOP-20_L6.5-W4.4-P0.65-LS6.4-BL, symbol EasyEDA:CH32V003F4P6
- added C11: 1 nF, Capacitor_SMD:C_0805_2012Metric_Pad1.18x1.45mm_HandSolder, symbol Device:C
- added CN2: B4B-PH-K-S, EasyEDA:CONN-TH_B6B-PH-K-S, symbol EasyEDA:B6B-PH-K-S
- added D1: BAT54SLT1G, EasyEDA:SOT-23_L2.9-W1.3-P1.90-LS2.4-BR, symbol EasyEDA:BAT54SLT1G
- added Q1: 2N7002, Package_TO_SOT_SMD:SOT-23, symbol Transistor_FET:2N7002
- added R10: 1k, Resistor_SMD:R_0805_2012Metric, symbol Device:R
- added R11: 200, Resistor_SMD:R_0805_2012Metric, symbol Device:R
- added R12: 1 k, Resistor_SMD:R_0805_2012Metric, symbol Device:R
- added TP2: TestPoint_2Pole, TestPoint:TestPoint_2Pads_Pitch2.54mm_Drill0.8mm, symbol Connector:TestPoint_2Pole
- added TP3, TP4, TP5, TP6: TestPoint, Connector_Pin:Pin_D0.7mm_L6.5mm_W1.8mm_FlatFork, symbol Connector:TestPoint
- added U5: CH32V103R8T6, EasyEDA:LQFP-64_L10.0-W10.0-P0.50-LS12.0-BL, symbol EasyEDA:CH32V103R8T6
- C1, C2, C3, C4, C5: footprint Capacitor_SMD:C_0805_2012Metric_Pad1.18x1.45mm_HandSolder -> Capacitor_SMD:C_0603_1608Metric
- C10: value 100 pF -> 100 nF
- C8: value 100 pF -> 1000 pF
- CN1: footprint EasyEDA:CONN-TH_B4B-PH-K-S -> EasyEDA:CONN-TH_B6B-PH-K-S; symbol EasyEDA:B4B-PH-K-S -> EasyEDA:B6B-PH-K-S; LCSC Part C131334 -> C131342; MPN B4B-PH-K-S(LF)(SN) -> B6B-PH-K-S(LF)(SN)
- R1: value 4.7 k -> 10 k; footprint Resistor_SMD:R_0805_2012Metric_Pad1.20x1.40mm_HandSolder -> Resistor_SMD:R_0805_2012Metric
- R2, R3, R4, R5, R6, R7, R8: footprint Resistor_SMD:R_0805_2012Metric_Pad1.20x1.40mm_HandSolder -> Resistor_SMD:R_0805_2012Metric
- R9: value 1 k -> 200; footprint Resistor_SMD:R_0805_2012Metric_Pad1.20x1.40mm_HandSolder -> Resistor_SMD:R_0805_2012Metric
- TP1: footprint (none) -> TestPoint:TestPoint_2Pads_Pitch2.54mm_Drill0.8mm
Connections:
- net +5V: now also CN2.1
- net GND: now also TP1.2, CN2.2, TP2.2
- net OUT_A: now also TP1.1
- net OUT_B: now also D1.1 (A), R12.1, TP2.1
- net PD3: now also TP5.1
- net SCL: no longer CN1.4
- net SDA: no longer CN1.3
- net v_half_ref: now also C11.2, D1.2 (C), Q1.2 (S), R10.1, TP3.1
- net at R7.2, R8.1, U4.1 (-IN): now also TP4.1
- new net: Q1.3 (D), R12.2
- new net PC3: Q1.1 (G)
- new net PD2: R11.1
- new net PD2 Pre: C11.1, D1.3 (A/C), R10.2, R11.2
- new net SENSOR_LP_0: U5.8 (PC0)
- new net SENSOR_LP_1: U5.9 (PC1)
- new net SENSOR_LP_10: U5.22 (PA6)
- new net SENSOR_LP_11: U5.23 (PA7)
- new net SENSOR_LP_12: U5.24 (PC4)
- new net SENSOR_LP_13: U5.25 (PC5)
- new net SENSOR_LP_14: U5.26 (PB0)
- new net SENSOR_LP_15: U5.27 (PB1)
- new net SENSOR_LP_2: U5.10 (PC2)
- new net SENSOR_LP_3: U5.11 (PC3)
- new net SENSOR_LP_4: U5.14 (PA0-WKUP)
- new net SENSOR_LP_5: U5.15 (PA1)
- new net SENSOR_LP_6: U5.16 (PA2)
- new net SENSOR_LP_7: U5.17 (PA3)
- new net SENSOR_LP_8: U5.20 (PA4)
- new net SENSOR_LP_9: U5.21 (PA5)
- new net SYS_SPI_MOSI: CN1.5, CN2.5
- new net SYS_SPI_SCK: CN1.3, CN2.3
- no-connect marks 6 -> 3
Other:
- added sheet Op amps (amplification.kicad_sch)
- moved on the sheet: C10, R3, R5, R6, R7, R8, R9, TP1, U4
