File: cap_tracker_tx/cap_tracker_tx.kicad_pcb (KiCad board)
At the start: 0 parts

Commit message: finished preliminary drawing
Parts:
- added Battery1: B2B-PH-K-S, EasyEDA:CONN-TH_B2B-PH-K-S, F.Cu at (114.8, 70.9)
- added Boot1: TS-1187A-B-A-B, EasyEDA:SW-SMD_4P-L5.1-W5.1-P3.70-LS6.5-TL_H1.5, F.Cu at (161.4, 72.8)
- added C1: 100 nF, Capacitor_SMD:C_0805_2012Metric_Pad1.18x1.45mm_HandSolder, F.Cu at (140.2, 76.2)
- added C2: 100 nF, Capacitor_SMD:C_0805_2012Metric_Pad1.18x1.45mm_HandSolder, F.Cu at (135.8, 55.0)
- added C3: 10 uF, Capacitor_SMD:C_0805_2012Metric_Pad1.18x1.45mm_HandSolder, F.Cu at (109.0, 67.5)
- added C4: 100 nF, Capacitor_SMD:C_0805_2012Metric_Pad1.18x1.45mm_HandSolder, F.Cu at (151.8, 83.0)
- added C5: 10 uF, Capacitor_SMD:C_0805_2012Metric_Pad1.18x1.45mm_HandSolder, F.Cu at (114.8, 59.4)
- added C6: 1 uF, Capacitor_SMD:C_0805_2012Metric_Pad1.18x1.45mm_HandSolder, F.Cu at (125.5, 53.2)
- added C7: 100 nF, Capacitor_SMD:C_0805_2012Metric_Pad1.18x1.45mm_HandSolder, F.Cu at (160.8, 88.7)
- added C8: 220 nF, Capacitor_SMD:C_0805_2012Metric_Pad1.18x1.45mm_HandSolder, F.Cu at (143.5, 71.5)
- added CN1: YZ182615065D-01, EasyEDA:SMD-1_BD2.0-D1.0, B.Cu at (165.2, 89.3)
- added EN1: TS-1187A-B-A-B, EasyEDA:SW-SMD_4P-L5.1-W5.1-P3.70-LS6.5-TL_H1.5, F.Cu at (126.2, 58.5)
- added JP1: Jumper_2_Small_Bridged, Panelization:MouseBite-Slot-Jumper_01005, F.Cu at (108.1, 62.2)
- added JP2: Jumper_2_Small_Bridged, Panelization:MouseBite-Slot-Jumper_01005, F.Cu at (108.1, 64.5)
- added LEDG1: YLED0603G, EasyEDA:LED0603-FD, F.Cu at (131.4, 64.9)
- added LEDR1: YLED0603R, EasyEDA:LED0603-FD, F.Cu at (131.6, 62.9)
- added Q1: AO3401A_C347476, EasyEDA:SOT-23_L2.9-W1.3-P1.90-LS2.4-BR, F.Cu at (115.7, 77.7)
- added Q2: MMBT3904LT1G, EasyEDA:SOT-23-3_L2.9-W1.6-P1.90-LS2.8-BR, F.Cu at (111.7, 81.6)
- added Q3: AO3401A_C347476, EasyEDA:SOT-23_L2.9-W1.3-P1.90-LS2.4-BR, F.Cu at (116.2, 82.4)
- added R1: 5.1k, Resistor_SMD:R_0805_2012Metric_Pad1.20x1.40mm_HandSolder, F.Cu at (159.5, 61.2)
- added R10: 10K, Resistor_SMD:R_0805_2012Metric_Pad1.20x1.40mm_HandSolder, F.Cu at (128.3, 53.3)
- added R11: 2.2K, Resistor_SMD:R_0805_2012Metric_Pad1.20x1.40mm_HandSolder, F.Cu at (141.7, 67.3)
- added R12: 2.2K, Resistor_SMD:R_0805_2012Metric_Pad1.20x1.40mm_HandSolder, F.Cu at (146.7, 66.6)
- added R13: 2.4K, Resistor_SMD:R_0805_2012Metric_Pad1.20x1.40mm_HandSolder, F.Cu at (104.8, 62.2)
- added R14: 100K, Resistor_SMD:R_0805_2012Metric_Pad1.20x1.40mm_HandSolder, F.Cu at (114.0, 85.0)
- added R15: 100K, Resistor_SMD:R_0805_2012Metric_Pad1.20x1.40mm_HandSolder, F.Cu at (106.5, 78.7)
- added R16: 1.2K, Resistor_SMD:R_0805_2012Metric_Pad1.20x1.40mm_HandSolder, F.Cu at (104.8, 64.5)
- added R17: HNTC-103F3950FB, EasyEDA:RES-TH_BD2.5-P2.0_HNTC-103F3950FB, F.Cu at (112.8, 55.5)
- added R2: 5.1k, Resistor_SMD:R_0805_2012Metric_Pad1.20x1.40mm_HandSolder, F.Cu at (159.5, 56.5)
- added R3: 100K, Resistor_SMD:R_0805_2012Metric_Pad1.20x1.40mm_HandSolder, F.Cu at (110.0, 59.4)
- added R4: 100K, Resistor_SMD:R_0805_2012Metric_Pad1.20x1.40mm_HandSolder, F.Cu at (110.8, 78.7)
- added R5: 100K, Resistor_SMD:R_0805_2012Metric_Pad1.20x1.40mm_HandSolder, F.Cu at (117.2, 86.0)
- added R6: 10K, Resistor_SMD:R_0805_2012Metric_Pad1.20x1.40mm_HandSolder, F.Cu at (106.5, 80.9)
- added R8: 1K, Resistor_SMD:R_0805_2012Metric_Pad1.20x1.40mm_HandSolder, F.Cu at (126.8, 62.9)
- added R9: 470, Resistor_SMD:R_0805_2012Metric_Pad1.20x1.40mm_HandSolder, F.Cu at (126.8, 64.9)
- added U1: 74LVC1G08GW_C52140431, EasyEDA:SOT-353-5_L2.1-W1.3-P0.65-LS2.3-BL, F.Cu at (159.8, 83.3)
- added U2: TP4056, EasyEDA:ESOP-8_L4.9-W3.9-P1.27-LS6.0-BL-EP, F.Cu at (114.8, 63.9)
- added U3: AP2112K-3.3TRG1_C23380830, EasyEDA:SOT-23-5_L2.9-W1.6-P0.95-LS2.8-BR, F.Cu at (120.7, 79.8)
- added U4: ESP32-C3-MINI-1-N4, EasyEDA:WIFIM-SMD_ESP32-C3-MINI-1, F.Cu at (146.5, 56.4)
- added U5: LIS2MDLTR, EasyEDA:VLGA-12_L2.0-W2.0-P0.50-BL, F.Cu at (146.2, 69.8)
- added U6: LSM6DSOXTR, EasyEDA:LGA-14L_L3.0-W2.5-P0.50-TL, F.Cu at (145.6, 75.5)
- added USB1: TYPE-C 16PIN 2MD, EasyEDA:USB-C-SMD_TYPE-C-16PIN-2MD-073, F.Cu at (167.7, 59.2)
- added X2: SX3M13.560B10F20TNN, EasyEDA:OSC-SMD_4P-L3.2-W2.5-BL-1, F.Cu at (156.0, 83.8)
Routing:
- net +3.3V: track 0.00 -> 83.3 mm, vias 0 -> 3
- net Batt Level: track 0.00 -> 46.9 mm, vias 0 -> 2
- net GND: track 0.00 -> 44.0 mm, vias 0 -> 23
- net USB 5V: track 0.00 -> 33.1 mm, vias 0 -> 10
- net IBC Modulation: track 0.00 -> 30.6 mm, vias 0 -> 2
- net Net-(Q1-S): track 0.00 -> 30.2 mm
- net SDA: track 0.00 -> 23.6 mm
- net EN: track 0.00 -> 21.3 mm
- net SCL: track 0.00 -> 20.3 mm
- net Boot: track 0.00 -> 18.9 mm
- net IMU Interrupt: track 0.00 -> 16.6 mm, vias 0 -> 2
- net Dn: track 0.00 -> 15.8 mm
- net Dp: track 0.00 -> 15.7 mm
- net Net-(U2-TEMP): track 0.00 -> 10.5 mm
- net /ENIG Surface: track 0.00 -> 9.69 mm, vias 0 -> 1
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- added copper zone on B.Cu, net /ENIG Surface
- added copper zone on F.Cu, net GND
- added copper zone on In1.Cu, net GND
- added copper zone on In2.Cu, net USB 5V
Other:
- board outline added: 71.8 x 40.5 mm
- copper layers 0 -> 4

Commit message: Modular Design
Parts:
- moved CN1 26.1 mm to (139.5, 84.5), turned to -90 degrees
- moved C7 17.3 mm to (144.0, 84.5), turned to 180 degrees
- moved U1 14.1 mm to (146.2, 86.8), turned to 90 degrees
- moved X2 6.60 mm to (149.9, 86.2), turned to 180 degrees
- moved C4 4.73 mm to (154.2, 87.1), turned to 180 degrees
Routing:
- net /ENIG Surface: track 9.69 -> 0.00 mm
- net Net-(U1-Y): track 3.73 -> 1.67 mm
- net IBC Modulation: track 30.6 -> 31.2 mm
Other:
- board text added: "Contact zone for children"
- board text added: "Design by JohnGF Version 1.0"
