File: cap_tracker_tx/cap_tracker_tx.kicad_sch (KiCad schematic)
At the start: 39 parts, among them CN1 YZ182615065D-01, Q1 AO3401A_C347476, Q2 MMBT3904LT1G, Q3 AO3401A_C347476, U1 74LVC1G08GW_C52140431, U2 TP4056, U3 AP2112K-3.3TRG1_C23380830, U4 ESP32-C3-MINI-1-N4, X2 SX3M13.560B10F20TNN

Commit message: finished preliminary drawing
Parts:
- C2, C3, C4, C5, C6, C7: footprint (none) -> Capacitor_SMD:C_0805_2012Metric_Pad1.18x1.45mm_HandSolder
- JP1, JP2: footprint (none) -> Panelization:MouseBite-Slot-Jumper_01005
- R1, R10, R11, R12, R13, R14, R15, R16, R2, R3, R4, R5, R6, R8, R9: footprint (none) -> Resistor_SMD:R_0805_2012Metric_Pad1.20x1.40mm_HandSolder
Connections:
- net +5V is gone; now on net USB 5V: C3.1, LEDG1.1 (+), LEDR1.1 (+), U2.4 (VCC), U2.8 (CE), USB1.A4B9 (VBUS), USB1.B4A9 (VBUS)
- net GND: now also USB1.13 (EH), USB1.14 (EH)

Commit message: Modular Design
Parts:
- removed Battery1: B2B-PH-K-S, EasyEDA:CONN-TH_B2B-PH-K-S, symbol EasyEDA:B2B-PH-K-S
- removed Boot1, EN1: TS-1187A-B-A-B, EasyEDA:SW-SMD_4P-L5.1-W5.1-P3.70-LS6.5-TL_H1.5, symbol EasyEDA:TS-1187A-B-A-B
- removed C2, C4, C7: 100 nF, Capacitor_SMD:C_0805_2012Metric_Pad1.18x1.45mm_HandSolder, symbol Device:C
- removed C3, C5: 10 uF, Capacitor_SMD:C_0805_2012Metric_Pad1.18x1.45mm_HandSolder, symbol Device:C
- removed C6: 1 uF, Capacitor_SMD:C_0805_2012Metric_Pad1.18x1.45mm_HandSolder, symbol Device:C
- removed CN1: YZ182615065D-01, EasyEDA:SMD-1_BD2.0-D1.0, symbol EasyEDA:YZ182615065D-01
- removed JP1, JP2: Jumper_2_Small_Bridged, Panelization:MouseBite-Slot-Jumper_01005, symbol Jumper:Jumper_2_Small_Bridged
- removed LEDG1: YLED0603G, EasyEDA:LED0603-FD, symbol EasyEDA:YLED0603G
- removed LEDR1: YLED0603R, EasyEDA:LED0603-FD, symbol EasyEDA:YLED0603R
- removed Q1, Q3: AO3401A_C347476, EasyEDA:SOT-23_L2.9-W1.3-P1.90-LS2.4-BR, symbol EasyEDA:AO3401A_C347476
- removed Q2: MMBT3904LT1G, EasyEDA:SOT-23-3_L2.9-W1.6-P1.90-LS2.8-BR, symbol EasyEDA:MMBT3904LT1G
- removed R1, R2: 5.1k, Resistor_SMD:R_0805_2012Metric_Pad1.20x1.40mm_HandSolder, symbol Device:R
- removed R10, R6: 10K, Resistor_SMD:R_0805_2012Metric_Pad1.20x1.40mm_HandSolder, symbol Device:R
- removed R11, R12: 2.2K, Resistor_SMD:R_0805_2012Metric_Pad1.20x1.40mm_HandSolder, symbol Device:R
- removed R13: 2.4K, Resistor_SMD:R_0805_2012Metric_Pad1.20x1.40mm_HandSolder, symbol Device:R
- removed R14, R15, R3, R4, R5: 100K, Resistor_SMD:R_0805_2012Metric_Pad1.20x1.40mm_HandSolder, symbol Device:R
- removed R16: 1.2K, Resistor_SMD:R_0805_2012Metric_Pad1.20x1.40mm_HandSolder, symbol Device:R
- removed R17: HNTC-103F3950FB, EasyEDA:RES-TH_BD2.5-P2.0_HNTC-103F3950FB, symbol EasyEDA:HNTC-103F3950FB
- removed R8: 1K, Resistor_SMD:R_0805_2012Metric_Pad1.20x1.40mm_HandSolder, symbol Device:R
- removed R9: 470, Resistor_SMD:R_0805_2012Metric_Pad1.20x1.40mm_HandSolder, symbol Device:R
- removed U1: 74LVC1G08GW_C52140431, EasyEDA:SOT-353-5_L2.1-W1.3-P0.65-LS2.3-BL, symbol EasyEDA:74LVC1G08GW_C52140431
- removed U2: TP4056, EasyEDA:ESOP-8_L4.9-W3.9-P1.27-LS6.0-BL-EP, symbol EasyEDA:TP4056
- removed U3: AP2112K-3.3TRG1_C23380830, EasyEDA:SOT-23-5_L2.9-W1.6-P0.95-LS2.8-BR, symbol EasyEDA:AP2112K-3.3TRG1_C23380830
- removed U4: ESP32-C3-MINI-1-N4, EasyEDA:WIFIM-SMD_ESP32-C3-MINI-1, symbol EasyEDA:ESP32-C3-MINI-1-N4
- removed USB1: TYPE-C 16PIN 2MD, EasyEDA:USB-C-SMD_TYPE-C-16PIN-2MD-073, symbol EasyEDA:TYPE-C16PIN2MD
- removed X2: SX3M13.560B10F20TNN, EasyEDA:OSC-SMD_4P-L3.2-W2.5-BL-1, symbol EasyEDA:SX3M13.560B10F20TNN
Connections:
- no-connect marks 17 -> 0
Other:
- sheet IMU renamed Signal
- added sheet Power (power.kicad_sch)
- sheet Signal: file imu.kicad_sch -> signal.kicad_sch
- note removed: "1.2K = 1A charge rate"
- note removed: "Cristal OOK Driving"
- note removed: "I2C BUS"
