File: cap_tracker_tx/imu.kicad_sch (KiCad schematic)
At the start: 4 parts, among them U5 LIS2MDLTR, U6 LSM6DSOXTR

Commit message: finished preliminary drawing
Parts:
- C1, C8: footprint (none) -> Capacitor_SMD:C_0805_2012Metric_Pad1.18x1.45mm_HandSolder

Commit message: Modular Design
Parts:
- removed C1: 100 nF, Capacitor_SMD:C_0805_2012Metric_Pad1.18x1.45mm_HandSolder, symbol Device:C
- added C12: 100 nF, Capacitor_SMD:C_0805_2012Metric_Pad1.18x1.45mm_HandSolder, symbol Device:C
- renumbered C8 to C13, U6 to U12, U5 to U13
Connections:
- net +3.3V: now also C13.2, C12.1; no longer U12.1 (SDO/SA0), U12.12 (CS), U12.5 (VDDIO), U13.3 (CS)
- net GND: now also C12.2
- net IMU Interrupt: now also U12.12 (CS); no longer U12.4 (INT1)
- net at U13.5 (C1): no longer C13.2
- net SCL renamed I2C_SYS.SCL
- net SDA renamed I2C_SYS.SDA
- new net Mag_interrupt: U13.3 (CS)
- no-connect marks 8 -> 3
Other:
- note added: "CS=VCC select I2Cn"
- note removed: "CS=VCC select I2C"
- moved on the sheet: C13, U13
